File: pcb/amtdoor3.sch (KiCad schematic (older format))
At the start: 76 parts, among them P1 CONN_01X04, P2 CONN_01X04, P3 CONN_01X04, P4 dnp-REF-182665-01, P5 CONN_01X02, P6 CONN_01X02, Q1 Q_NMOS_DUAL, Q10 Q_NMOS_DUAL, Q2 Q_PMOS_HP, Q3 DMMT3906_Dual_PNP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

Commit message: update bom info for pcb rev 2.0
Parts:
- Q1: Description (none) -> MOSFET 2N-CH 50V 0.305A SOT-26; Digikey Part No (none) -> DMN5L06DMKDICT-ND; Mfg (none) -> Diodes Inc; Mfg Part No (none) -> DMN5L06DMK-7; Type (none) -> SMT
- Q10, Q5, Q6, Q7, Q8, Q9: Mfg (none) -> Diodes Inc; Mfg Part No (none) -> DMN5L06DMK-7
- U3: Digikey Part No todo -> 296-39451-1-ND; Mfg Part No todo -> TPS62175DQCR
Changed lines of the file:
@@
 encoding utf-8
 Sheet 1 1
-Title "AMT Door 3 - RPi Zero IO"
-Date "2016-10-16"
-Rev "1.0"
+Title "Wide Operation Buck Boost and Automation pHat (WOBBApHAT)"
+Date "2017-09-25"
+Rev "2.0"
 Comp ""
 Comment1 "Author: Ian Hartwig"
 Comment2 "License: CERN OHL V1.2"
-Comment3 ""
+Comment3 "HW for AMT Door 3"
 Comment4 ""
 $EndDescr
@@
 F 3 "" H 7900 7950 50  0000 C CNN
 F 4 "Diodes Inc" H 7900 7950 60  0001 C CNN "Mfg"
-F 5 "DMG4435SSS-13" H 7900 7950 60  0001 C CNN "Mfg Part No"
+F 5 "DMG4435SSS-13" H 8650 8000 60  0000 C CNN "Mfg Part No"
 F 6 "DMG4435SSS-13DICT-ND" H 7900 7950 60  0001 C CNN "Digikey Part No"
 F 7 "MOSFET P-CH 30V 7.3A 8SOIC" H 7900 7950 60  0001 C CNN "Description"
@@
 F 3 "" H 2800 10150 60  0000 C CNN
 F 4 "Texas Instruments" H 2800 10150 60  0001 C CNN "Mfg"
-F 5 "todo" H 2800 10150 60  0001 C CNN "Mfg Part No"
-F 6 "todo" H 2800 10150 60  0001 C CNN "Digikey Part No"
+F 5 "TPS62175DQCR" H 2800 10150 60  0001 C CNN "Mfg Part No"
+F 6 "296-39451-1-ND" H 2800 10150 60  0001 C CNN "Digikey Part No"
 F 7 "Buck Switching Regulator IC Positive Fixed 3.3V 1 Output 500mA 10-WFDFN Exposed Pad" H 2800 10150 60  0001 C CNN "Description"
 F 8 "SMT" H 2800 10150 60  0001 C CNN "Type"
@@
 F 3 "" H 4050 9950 50  0000 C CNN
 F 4 "Taiyo Yuden" H 4050 9950 60  0001 C CNN "Mfg"
-F 5 "NR6045T100M" H 4050 9950 60  0001 C CNN "Mfg Part No"
+F 5 "NR6045T100M" H 4050 10150 60  0000 C CNN "Mfg Part No"
 F 6 "587-2081-1-ND" H 4050 9950 60  0001 C CNN "Digikey Part No"
 F 7 "10µH Shielded Wirewound Inductor 2.5A 61.1 mOhm Max Nonstandard" H 4050 9950 60  0001 C CNN "Description"
@@
 F 3 "" H 6600 10250 50  0000 C CNN
 F 4 "Diodes Inc" H 6450 10250 60  0001 C CNN "Mfg"
-F 5 "DMMT3906-7-F" H 6450 10250 60  0001 C CNN "Mfg Part No"
+F 5 "DMMT3906-7-F" H 7350 10300 60  0000 C CNN "Mfg Part No"
 F 6 "DMMT3906-7-FDICT-ND" H 6450 10250 60  0001 C CNN "Digikey Part No"
 F 7 "SMT" H 6450 10250 60  0001 C CNN "Type"
@@
 F 3 "" H 6500 9850 50  0000 C CNN
 F 4 "Diodes Inc" H 6500 9850 60  0001 C CNN "Mfg"
-F 5 "DMP3099L-7" H 6500 9850 60  0001 C CNN "Mfg Part No"
+F 5 "DMP3099L-7" H 7150 9900 60  0000 C CNN "Mfg Part No"
 F 6 "DMP3099L-7DICT-ND" H 6500 9850 60  0001 C CNN "Digikey Part No"
 F 7 "SMT" H 6500 9850 60  0001 C CNN "Type"
@@
 F 2 "TO_SOT_Packages_SMD:SOT-23-6" H 7500 8450 50  0001 C CNN
 F 3 "" H 7300 8350 50  0000 C CNN
+F 4 "Diodes Inc" H 7300 8350 60  0001 C CNN "Mfg"
+F 5 "DMN5L06DMK-7" H 7300 8350 60  0001 C CNN "Mfg Part No"
+F 6 "MOSFET 2N-CH 50V 0.305A SOT-26" H 7300 8350 60  0001 C CNN "Description"
+F 7 "DMN5L06DMKDICT-ND" H 7300 8350 60  0001 C CNN "Digikey Part No"
+F 8 "SMT" H 7300 8350 60  0001 C CNN "Type"
 	1    7300 8350
 	1    0    0    -1
@@
 F 2 "TO_SOT_Packages_SMD:SOT-23-6" H 9700 8450 50  0001 C CNN
 F 3 "" H 9500 8350 50  0000 C CNN
+F 4 "Diodes Inc" H 9500 8350 60  0001 C CNN "Mfg"
+F 5 "DMN5L06DMK-7" H 9500 8350 60  0001 C CNN "Mfg Part No"
+F 6 "MOSFET 2N-CH 50V 0.305A SOT-26" H 9500 8350 60  0001 C CNN "Description"
+F 7 "SMT" H 9500 8350 60  0001 C CNN "Type"
+F 8 "DMN5L06DMKDICT-ND" H 9500 8350 60  0001 C CNN "Digikey Part No"
 	2    9500 8350
 	1    0    0    -1
@@
 	2300 10050 2200 10050
 Wire Wire Line
-	2200 9950 2200 10050
+	2200 10050 2200 9950
 Connection ~ 2200 9950
 Wire Wire Line
@@
 	6300 9750 6100 9750
 Wire Wire Line
-	6100 9950 6100 9750
+	6100 9750 6100 9950
 Connection ~ 6100 9950
 Wire Wire Line
@@
 F 2 "TO_SOT_Packages_SMD:SOT-23-6" H 2900 5700 50  0001 C CNN
 F 3 "" H 2700 5600 50  0000 C CNN
+F 4 "Diodes Inc" H 2700 5600 60  0001 C CNN "Mfg"
+F 5 "DMN5L06DMK-7" H 2700 5600 60  0001 C CNN "Mfg Part No"
 	2    2700 5600
 	0    1    1    0
@@
 F 2 "TO_SOT_Packages_SMD:SOT-23-6" H 3300 5300 50  0001 C CNN
 F 3 "" H 3100 5200 50  0000 C CNN
+F 4 "Diodes Inc" H 3100 5200 60  0001 C CNN "Mfg"
+F 5 "DMN5L06DMK-7" H 3100 5200 60  0001 C CNN "Mfg Part No"
 	1    3100 5200
 	0    1    1    0
@@
 F 2 "TO_SOT_Packages_SMD:SOT-23-6" H 7100 5900 50  0001 C CNN
 F 3 "" H 6900 5800 50  0000 C CNN
+F 4 "Diodes Inc" H 6900 5800 60  0001 C CNN "Mfg"
+F 5 "DMN5L06DMK-7" H 6900 5800 60  0001 C CNN "Mfg Part No"
 	1    6900 5800
 	1    0    0    -1
@@
 F 2 "TO_SOT_Packages_SMD:SOT-23-6" H 8700 5900 50  0001 C CNN
 F 3 "" H 8500 5800 50  0000 C CNN
+F 4 "Diodes Inc" H 8500 5800 60  0001 C CNN "Mfg"
+F 5 "DMN5L06DMK-7" H 8500 5800 60  0001 C CNN "Mfg Part No"
 	2    8500 5800
 	1    0    0    -1
@@
 F 2 "TO_SOT_Packages_SMD:SOT-23-6" H 2900 3800 50  0001 C CNN
 F 3 "" H 2700 3700 50  0000 C CNN
+F 4 "Diodes Inc" H 2700 3700 60  0001 C CNN "Mfg"
+F 5 "DMN5L06DMK-7" H 2700 3700 60  0001 C CNN "Mfg Part No"
 	2    2700 3700
 	0    1    1    0
@@
 F 2 "TO_SOT_Packages_SMD:SOT-23-6" H 3300 3400 50  0001 C CNN
 F 3 "" H 3100 3300 50  0000 C CNN
+F 4 "Diodes Inc" H 3100 3300 60  0001 C CNN "Mfg"
+F 5 "DMN5L06DMK-7" H 3100 3300 60  0001 C CNN "Mfg Part No"
 	1    3100 3300
 	0    1    1    0
@@
 F 2 "TO_SOT_Packages_SMD:SOT-23-6" H 7100 4000 50  0001 C CNN
 F 3 "" H 6900 3900 50  0000 C CNN
+F 4 "Diodes Inc" H 6900 3900 60  0001 C CNN "Mfg"
+F 5 "DMN5L06DMK-7" H 6900 3900 60  0001 C CNN "Mfg Part No"
 	1    6900 3900
 	1    0    0    -1
@@
 F 2 "TO_SOT_Packages_SMD:SOT-23-6" H 8700 4000 50  0001 C CNN
 F 3 "" H 8500 3900 50  0000 C CNN
+F 4 "Diodes Inc" H 8500 3900 60  0001 C CNN "Mfg"
+F 5 "DMN5L06DMK-7" H 8500 3900 60  0001 C CNN "Mfg Part No"
 	2    8500 3900
 	1    0    0    -1
@@
 F 2 "TO_SOT_Packages_SMD:SOT-23-6" H 2900 1900 50  0001 C CNN
 F 3 "" H 2700 1800 50  0000 C CNN
+F 4 "Diodes Inc" H 2700 1800 60  0001 C CNN "Mfg"
+F 5 "DMN5L06DMK-7" H 2700 1800 60  0001 C CNN "Mfg Part No"
 	2    2700 1800
 	0    1    1    0
@@
 F 2 "TO_SOT_Packages_SMD:SOT-23-6" H 3300 1500 50  0001 C CNN
 F 3 "" H 3100 1400 50  0000 C CNN
+F 4 "Diodes Inc" H 3100 1400 60  0001 C CNN "Mfg"
+F 5 "DMN5L06DMK-7" H 3100 1400 60  0001 C CNN "Mfg Part No"
 	1    3100 1400
 	0    1    1    0
@@
 F 2 "TO_SOT_Packages_SMD:SOT-23-6" H 7100 2100 50  0001 C CNN
 F 3 "" H 6900 2000 50  0000 C CNN
+F 4 "Diodes Inc" H 6900 2000 60  0001 C CNN "Mfg"
+F 5 "DMN5L06DMK-7" H 6900 2000 60  0001 C CNN "Mfg Part No"
 	1    6900 2000
 	1    0    0    -1
@@
 F 2 "TO_SOT_Packages_SMD:SOT-23-6" H 8700 2100 50  0001 C CNN
 F 3 "" H 8500 2000 50  0000 C CNN
+F 4 "Diodes Inc" H 8500 2000 60  0001 C CNN "Mfg"
+F 5 "DMN5L06DMK-7" H 8500 2000 60  0001 C CNN "Mfg Part No"
 	2    8500 2000
 	1    0    0    -1
